File: Hardware/Waage/Waage.kicad_pcb (KiCad board)
At the start: 2 copper layers, 70 x 62.5 mm, 59 parts, among them J1 USB_B, J2 Conn_01x04_Female, J3 Conn_01x04_Female, J4 Conn_01x04_Female, SW1 SW_Push, SW2 SW_Push, SW3 SW_Push, SW4 SW_Push, SW5 SW_Push, U1 USBLC6-2SC6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

Commit message: update CAD + Layout
Parts:
- added BT1: Battery_Cell, Battery:BatteryHolder_Keystone_3000_1x12mm, F.Cu at (95.2, 76.7)
- added U9: PCF8563T, Package_SO:SOIC-8_3.9x4.9mm_P1.27mm, F.Cu at (104.5, 68.0)
- moved R4 6.17 mm to (102.6, 85.1), turned to 270 degrees
- moved C8 3.90 mm to (108.7, 73.3), turned to 90 degrees
Routing:
- net Net-(BT1-Pad2): track 0.00 -> 28.1 mm
- net Net-(BT1-Pad1): track 0.00 -> 12.7 mm
- net SDA: track 34.0 -> 46.5 mm
- net SCL: track 29.6 -> 41.0 mm
- net +3V3: track 157.6 -> 162.8 mm
- net GND: track 68.7 -> 67.8 mm, vias 15 -> 14
- net VDDA: track 71.5 -> 70.7 mm

Commit message: update layout
Parts:
- added C16: 100n, Capacitor_SMD:C_0603_1608Metric, F.Cu at (106.4, 73.4)
- added D4: D_Schottky, Diode_SMD:D_0603_1608Metric, F.Cu at (99.8, 67.7)
Connections:
- U9 pad 8: Net-(BT1-Pad1) -> +3V3
Routing:
- net Net-(BT1-Pad1): track 12.7 -> 4.25 mm
- net +3V3: track 162.8 -> 171.0 mm
- net GND: track 67.8 -> 70.1 mm
Changed lines of the file:
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@@
     (thickness 1.6)
     (drawings 5)
-    (tracks 662)
+    (tracks 668)
     (zones 0)
-    (modules 61)
+    (modules 63)
     (nets 52)
   )
@@
   )
   (setup
-    (last_trace_width 0.3)
+    (last_trace_width 0.25)
     (user_trace_width 0.3)
     (user_trace_width 0.4)
@@
     (visible_elements 7FFFFFFF)
     (pcbplotparams
-      (layerselection 0x010fc_ffffffff)
+      (layerselection 0x010cc_ffffffff)
       (usegerberextensions false)
       (usegerberattributes false)
@@
       (outputformat 1)
       (mirror false)
-      (drillshape 1)
+      (drillshape 0)
       (scaleselection 1)
-      (outputdirectory ""))
+      (outputdirectory "Fabrication/"))
   )
   (net 0 "")
@@
     (add_net VDDA)
   )
+  (module Diode_SMD:D_0603_1608Metric (layer F.Cu)
+    (at 99.85 67.7 180)
+    (descr "Diode SMD 0603 (1608 Metric), square (rectangular) end terminal, IPC_7351 nominal, (Body size source: http://www.tortai-tech.com/upload/download/2011102023233369053.pdf), generated with kicad-footprint-generator")
+    (tags diode)
+    (attr smd)
+    (fp_text reference D4 (at 0 -1.43 180) (layer F.SilkS)
+      (effects (font (size 1 1) (thickness 0.15)))
+    )
+    (fp_text value D_Schottky (at 0 1.43 180) (layer F.Fab)
+      (effects (font (size 1 1) (thickness 0.15)))
+    )
+    (fp_text user %R (at 0 0 180) (layer F.Fab)
+      (effects (font (size 0.4 0.4) (thickness 0.06)))
+    )
+    (fp_line (start 1.48 0.73) (end -1.48 0.73) (layer F.CrtYd) (width 0.05))
+    (fp_line (start 1.48 -0.73) (end 1.48 0.73) (layer F.CrtYd) (width 0.05))
+    (fp_line (start -1.48 -0.73) (end 1.48 -0.73) (layer F.CrtYd) (width 0.05))
+    (fp_line (start -1.48 0.73) (end -1.48 -0.73) (layer F.CrtYd) (width 0.05))
+    (fp_line (start -1.485 0.735) (end 0.8 0.735) (layer F.SilkS) (width 0.12))
+    (fp_line (start -1.485 -0.735) (end -1.485 0.735) (layer F.SilkS) (width 0.12))
+    (fp_line (start 0.8 -0.735) (end -1.485 -0.735) (layer F.SilkS) (width 0.12))
+    (fp_line (start 0.8 0.4) (end 0.8 -0.4) (layer F.Fab) (width 0.1))
+    (fp_line (start -0.8 0.4) (end 0.8 0.4) (layer F.Fab) (width 0.1))
+    (fp_line (start -0.8 -0.1) (end -0.8 0.4) (layer F.Fab) (width 0.1))
+    (fp_line (start -0.5 -0.4) (end -0.8 -0.1) (layer F.Fab) (width 0.1))
+    (fp_line (start 0.8 -0.4) (end -0.5 -0.4) (layer F.Fab) (width 0.1))
+    (pad 2 smd roundrect (at 0.7875 0 180) (size 0.875 0.95) (layers F.Cu F.Paste F.Mask) (roundrect_rratio 0.25)
+      (net 50 "Net-(BT1-Pad1)"))
+    (pad 1 smd roundrect (at -0.7875 0 180) (size 0.875 0.95) (layers F.Cu F.Paste F.Mask) (roundrect_rratio 0.25)
+      (net 4 +3V3))
+    (model ${KISYS3DMOD}/Diode_SMD.3dshapes/D_0603_1608Metric.wrl
+      (at (xyz 0 0 0))
+      (scale (xyz 1 1 1))
+      (rotate (xyz 0 0 0))
+    )
+  )
+  (module Capacitor_SMD:C_0603_1608Metric (layer F.Cu)
+    (at 106.4 73.4 270)
+    (descr "Capacitor SMD 0603 (1608 Metric), square (rectangular) end terminal, IPC_7351 nominal, (Body size source: http://www.tortai-tech.com/upload/download/2011102023233369053.pdf), generated with kicad-footprint-generator")
+    (tags capacitor)
+    (attr smd)
+    (fp_text reference C16 (at 0 -1.43 270) (layer F.SilkS)
+      (effects (font (size 1 1) (thickness 0.15)))
+    )
+    (fp_text value 100n (at 0 1.43 270) (layer F.Fab)
+      (effects (font (size 1 1) (thickness 0.15)))
+    )
+    (fp_text user %R (at 0 0 270) (layer F.Fab)
+      (effects (font (size 0.4 0.4) (thickness 0.06)))
+    )
+    (fp_line (start 1.48 0.73) (end -1.48 0.73) (layer F.CrtYd) (width 0.05))
+    (fp_line (start 1.48 -0.73) (end 1.48 0.73) (layer F.CrtYd) (width 0.05))
+    (fp_line (start -1.48 -0.73) (end 1.48 -0.73) (layer F.CrtYd) (width 0.05))
+    (fp_line (start -1.48 0.73) (end -1.48 -0.73) (layer F.CrtYd) (width 0.05))
+    (fp_line (start -0.162779 0.51) (end 0.162779 0.51) (layer F.SilkS) (width 0.12))
+    (fp_line (start -0.162779 -0.51) (end 0.162779 -0.51) (layer F.SilkS) (width 0.12))
+    (fp_line (start 0.8 0.4) (end -0.8 0.4) (layer F.Fab) (width 0.1))
+    (fp_line (start 0.8 -0.4) (end 0.8 0.4) (layer F.Fab) (width 0.1))
+    (fp_line (start -0.8 -0.4) (end 0.8 -0.4) (layer F.Fab) (width 0.1))
+    (fp_line (start -0.8 0.4) (end -0.8 -0.4) (layer F.Fab) (width 0.1))
+    (pad 2 smd roundrect (at 0.7875 0 270) (size 0.875 0.95) (layers F.Cu F.Paste F.Mask) (roundrect_rratio 0.25)
+      (net 1 GND))
+    (pad 1 smd roundrect (at -0.7875 0 270) (size 0.875 0.95) (layers F.Cu F.Paste F.Mask) (roundrect_rratio 0.25)
+      (net 4 +3V3))
+    (model ${KISYS3DMOD}/Capacitor_SMD.3dshapes/C_0603_1608Metric.wrl
+      (at (xyz 0 0 0))
+      (scale (xyz 1 1 1))
+      (rotate (xyz 0 0 0))
+    )
+  )
   (module Resistor_SMD:R_1206_3216Metric (layer F.Cu)
     (at 105.75 78.975 90)
@@
     )
     (pad 8 smd rect (at 2.7 -1.905 270) (size 1.55 0.6) (layers F.Cu F.Paste F.Mask)
-      (net 50 "Net-(BT1-Pad1)"))
+      (net 4 +3V3))
     (pad 7 smd rect (at 2.7 -0.635 270) (size 1.55 0.6) (layers F.Cu F.Paste F.Mask))
     (pad 6 smd rect (at 2.7 0.635 270) (size 1.55 0.6) (layers F.Cu F.Paste F.Mask)
@@
   (segment (start 108.65 75.6) (end 108.15 76.1) (width 0.3) (layer F.Cu) (net 1))
   (via (at 108.65 75.6) (size 0.8) (drill 0.4) (layers F.Cu B.Cu) (net 1))
+  (segment (start 106.4 74.1875) (end 107.6125 74.1875) (width 0.25) (layer F.Cu) (net 1))
+  (segment (start 107.7125 74.0875) (end 108.65 74.0875) (width 0.25) (layer F.Cu) (net 1))
+  (segment (start 107.6125 74.1875) (end 107.7125 74.0875) (width 0.25) (layer F.Cu) (net 1))
   (segment (start 112.9875 76.3125) (end 113 76.325) (width 0.3) (layer F.Cu) (net 2))
   (segment (start 111 76.3125) (end 112.9875 76.3125) (width 0.3) (layer F.Cu) (net 2))
@@
   (segment (start 108.65 72.5125) (end 109.225 72.5125) (width 0.3) (layer F.Cu) (net 4))
   (segment (start 109.225 72.5125) (end 110.2375 73.525) (width 0.3) (layer F.Cu) (net 4))
+  (segment (start 100.6375 67.7) (end 105.4 67.7) (width 0.25) (layer F.Cu) (net 4))
+  (segment (start 106.355 68.655) (end 106.355 70.75) (width 0.25) (layer F.Cu) (net 4))
+  (segment (start 105.4 67.7) (end 106.355 68.655) (width 0.25) (layer F.Cu) (net 4))
   (segment (start 122.1825 66.095702) (end 122.1825 65.0957) (width 0.3) (layer F.Cu) (net 5))
   (segment (start 120.2775 70.4043) (end 120.2775 68.000702) (width 0.3) (layer F.Cu) (net 5))
@@
   (segment (start 132.84 74.2) (end 142.23 74.2) (width 0.4) (layer B.Cu) (net 49))
   (segment (start 131.63 75.41) (end 132.84 74.2) (width 0.4) (layer B.Cu) (net 49))
-  (segment (start 105.7 68.75) (end 106.355 69.405) (width 0.5) (layer F.Cu) (net 50))
-  (segment (start 95.25 68.75) (end 105.7 68.75) (width 0.5) (layer F.Cu) (net 50))
-  (segment (start 106.355 70.75) (end 106.355 69.405) (width 0.5) (layer F.Cu) (net 50))
+  (segment (start 98.2 67.7) (end 99.0625 67.7) (width 0.25) (layer F.Cu) (net 50))
+  (segment (start 95.25 68.75) (end 97.15 68.75) (width 0.25) (layer F.Cu) (net 50))
+  (segment (start 97.15 68.75) (end 98.2 67.7) (width 0.25) (layer F.Cu) (net 50))
   (segment (start 95.25 76.65) (end 90.8 76.65) (width 0.5) (layer F.Cu) (net 51))
   (segment (start 90.8 76.65) (end 89.9 75.75) (width 0.5) (layer F.Cu) (net 51))
