File: Hardware/Waage_v2/Waage.kicad_pcb (KiCad board)
At the start: 2 copper layers, 70 x 62.5 mm, 58 parts, among them J1 USB_B, J2 Conn_01x04_Female, J3 Conn_01x04_Female, J4 Conn_01x04_Female, SW1 SW_Push, SW2 SW_Push, SW3 SW_Push, SW4 SW_Push, SW5 SW_Push, U1 USBLC6-2SC6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

Commit message: Update layout
Parts:
- added Q1: BC856, Package_TO_SOT_SMD:SOT-23, F.Cu at (138.1, 83.0)
- added R17: 1.5k, Resistor_SMD:R_1206_3216Metric, F.Cu at (91.3, 89.0)
- added R18: 10k, Resistor_SMD:R_1206_3216Metric, F.Cu at (141.1, 82.4)
- added R19: 1.5k, Resistor_SMD:R_1206_3216Metric, F.Cu at (133.2, 82.5)
- added R20: 1.5k, Resistor_SMD:R_1206_3216Metric, F.Cu at (141.1, 87.0)
- moved R10 5.17 mm to (138.7, 87.1)
Connections:
- C13 pad 1: 3.5V -> Net-(C13-Pad1)
- RV1 pad 2: Net-(RV1-Pad2) -> Net-(R17-Pad1)
- U2 pad 26: (no net) -> LCD_LIGHT
- U4 pad 1: (no net) -> Net-(U4-Pad1)
- U4 pad 2: (no net) -> Net-(U4-Pad2)
- U5 pad 10: (no net) -> Net-(U5-Pad10)
- U5 pad 3: Net-(RV1-Pad2) -> Net-(R17-Pad2)
- U5 pad 7: (no net) -> Net-(U5-Pad7)
- U5 pad 8: (no net) -> Net-(U5-Pad8)
- U5 pad 9: (no net) -> Net-(U5-Pad9)
- U7 pad 2: 3.5V -> Net-(C13-Pad1)
- U8 pad 6: Net-(RV1-Pad2) -> Net-(R17-Pad2)
- U9 pad 1: (no net) -> Net-(U9-Pad1)
- U9 pad 2: (no net) -> Net-(U9-Pad2)
- U9 pad 3: (no net) -> Net-(U9-Pad3)
- U9 pad 7: (no net) -> Net-(U9-Pad7)
Routing:
- net Net-(RV1-Pad2): track 27.4 -> 0.00 mm, vias 1 -> 0
- net Net-(BT1-Pad1): track 4.25 -> 27.3 mm
- net Net-(R17-Pad2): track 0.00 -> 20.9 mm, vias 0 -> 2
- net LCD_LIGHT: track 0.00 -> 18.7 mm, vias 0 -> 2
- net +3V3: track 174.3 -> 192.0 mm
- net Net-(C13-Pad1): track 0.00 -> 15.7 mm
- net Net-(Q1-Pad1): track 0.00 -> 10.0 mm
- net Net-(R15-Pad1): track 12.9 -> 21.8 mm
- net GND: track 62.1 -> 68.5 mm
- net Net-(R10-Pad1): track 23.0 -> 17.4 mm
- net Net-(R17-Pad1): track 0.00 -> 3.35 mm
- net 3.5V: track 4.63 -> 6.73 mm
- net SCL: track 52.7 -> 50.8 mm

Commit message: HW ueberarbeitung
Parts:
- removed R2, R20: 1.5k, Resistor_SMD:R_1206_3216Metric
- removed U5: NHD-0212WH, MK_Footprints:NHD-0212WH
- added C6: 100n, Capacitor_SMD:C_0603_1608Metric, F.Cu at (109.8, 72.5)
- added D5: D_Schottky, Diode_SMD:D_0603_1608Metric, F.Cu at (109.0, 53.2)
- added Y1: Crystal, Crystal:Crystal_SMD_3215-2Pin_3.2x1.5mm, F.Cu at (112.6, 69.7)
- R17: value 1.5k -> 0
- moved R4 9.70 mm to (105.0, 75.7), turned to 90 degrees
- moved R3 3.64 mm to (107.3, 75.7)
- moved U9 3.25 mm to (107.6, 69.0), turned to 180 degrees
- moved C16 3.13 mm to (105.3, 72.5)
Connections:
- BT1 pad 2: Net-(BT1-Pad2) -> GND
- C16 pad 1: +3V3 -> Net-(C16-Pad1)
- D4 pad 1: +3V3 -> Net-(C16-Pad1)
- J1 pad 2: D- -> (no net)
- U1 pad 1: D+ -> (no net)
- U1 pad 2: GND -> (no net)
- U1 pad 3: D- -> (no net)
- U1 pad 4: DM -> (no net)
- U1 pad 6: DP -> (no net)
- U2 pad 21: DM -> (no net)
- U2 pad 22: DP -> (no net)
- U4 pad 1: Net-(U4-Pad1) -> (no net)
- U4 pad 2: Net-(U4-Pad2) -> (no net)
- U8 pad 1: Net-(R2-Pad2) -> GND
- U9 pad 3: Net-(U9-Pad3) -> (no net)
- U9 pad 4: Net-(BT1-Pad2) -> GND
- U9 pad 7: Net-(U9-Pad7) -> (no net)
- U9 pad 8: +3V3 -> Net-(C16-Pad1)
Routing:
- net (no net): track 0.00 -> 89.5 mm, vias 0 -> 5
- net DM: track 37.6 -> 0.00 mm, vias 2 -> 0
- net DP: track 37.3 -> 0.00 mm, vias 2 -> 0
- net Net-(BT1-Pad2): track 28.1 -> 0.00 mm
- net SCL: track 50.8 -> 26.3 mm, vias 3 -> 2
- net GND: track 68.5 -> 89.9 mm, vias 9 -> 8
- net Net-(C16-Pad1): track 0.00 -> 14.4 mm
- net SCK_L2: track 20.8 -> 6.93 mm
- net DATA_L2: track 19.9 -> 8.07 mm
- net SDA: track 55.7 -> 44.7 mm, vias 3 -> 2
- net D-: track 11.0 -> 0.00 mm
- net +3V3: track 192.0 -> 184.0 mm
- net Net-(C6-Pad2): track 0.00 -> 4.11 mm
- net Net-(R2-Pad2): track 3.42 -> 0.00 mm
- net Net-(U9-Pad2): track 0.00 -> 3.24 mm

Commit message: update hw
Parts:
- added U5: NHD-0212WH, MK_Footprints:NHD-0212WH, F.Cu at (115.0, 76.5)
Connections:
- R10 pad 1: Net-(R10-Pad1) -> (no net)
- U2 pad 2: LCD_RS -> (no net)
- U2 pad 25: DB3 -> (no net)
- U2 pad 3: LCD_RW -> (no net)
- U2 pad 31: DB2 -> (no net)
- U2 pad 6: LCD_E -> (no net)
- U2 pad 7: DB0 -> (no net)
- U2 pad 8: DB1 -> (no net)
Routing:
- net (no net): track 89.5 -> 212.5 mm, vias 5 -> 8
- net LCD_RS: track 18.6 -> 0.00 mm
- net DB2: track 18.1 -> 0.00 mm, vias 1 -> 0
- net LCD_RW: track 17.6 -> 0.00 mm
- net Net-(R10-Pad1): track 17.4 -> 0.00 mm, vias 1 -> 0
- net DB3: track 16.0 -> 0.00 mm, vias 1 -> 0
- net LCD_E: track 12.5 -> 0.00 mm
- net DB0: track 12.5 -> 0.00 mm
- net DB1: track 10.3 -> 0.00 mm

Commit message: update software
Parts:
- removed C4: 100n, Capacitor_SMD:C_0603_1608Metric
- removed R17: 0, Resistor_SMD:R_1206_3216Metric
- removed RV1: R_POT, Potentiometer_THT:Potentiometer_Vishay_T73YP_Vertical
- added J5: Conn_01x02_Female, Connector_PinHeader_2.54mm:PinHeader_1x02_P2.54mm_Vertical, F.Cu at (137.4, 109.9)
- added R2: 0, Resistor_SMD:R_1206_3216Metric, F.Cu at (134.3, 109.4)
- moved C14 15.7 mm to (105.7, 70.2), turned to 0 degrees
- moved D5 14.5 mm to (108.0, 67.6), turned to 90 degrees
- moved U4 11.8 mm to (116.1, 73.6)
- moved U8 11.8 mm to (106.0, 74.2), turned to 90 degrees
- moved C8 11.8 mm to (117.3, 78.1)
- moved R15 11.3 mm to (120.0, 70.4), turned to 90 degrees
- moved R4 9.79 mm to (112.3, 82.2), turned to 270 degrees
- moved R1 8.91 mm to (120.0, 80.4)
- moved C1 8.87 mm to (117.2, 81.8), turned to 180 degrees
- moved R19 8.41 mm to (141.6, 82.0), turned to 0 degrees
- moved R16 7.86 mm to (120.0, 75.1)
- moved R3 7.00 mm to (110.0, 82.2), turned to 270 degrees
- moved C5 6.92 mm to (122.2, 77.2)
- moved U2 6.73 mm to (126.7, 82.0)
- moved D4 6.60 mm to (106.5, 67.6), turned to 90 degrees
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Connections:
- net Net-(R17-Pad2) renamed KONTRAST
- J1 pad 1: VBUS -> Net-(J1-Pad1)
- J1 pad 2: (no net) -> D-
- R10 pad 1: (no net) -> Net-(R10-Pad1)
- U1 pad 1: (no net) -> D+
- U1 pad 2: (no net) -> GND
- U1 pad 3: (no net) -> D-
- U1 pad 4: (no net) -> DM
- U1 pad 6: (no net) -> DP
- U2 pad 2: (no net) -> LCD_RS
- U2 pad 21: (no net) -> DM
- U2 pad 22: (no net) -> DP
- U2 pad 25: (no net) -> DB3
- U2 pad 3: (no net) -> LCD_RW
- U2 pad 31: (no net) -> DB2
- U2 pad 6: (no net) -> LCD_E
- U2 pad 7: (no net) -> DB0
- U2 pad 8: (no net) -> DB1
- U5 pad 10: Net-(U5-Pad10) -> (no net)
- U5 pad 7: Net-(U5-Pad7) -> (no net)
- U5 pad 8: Net-(U5-Pad8) -> (no net)
- U5 pad 9: Net-(U5-Pad9) -> (no net)
Routing:
- net (no net): track 212.5 -> 0.00 mm, vias 8 -> 0
- net DP: track 0.00 -> 34.7 mm, vias 0 -> 2
- net DM: track 0.00 -> 33.3 mm, vias 0 -> 2
- net +3V3: track 184.0 -> 212.0 mm, vias 6 -> 8
- net SCL: track 26.3 -> 51.9 mm, vias 2 -> 3
- net SCK_L2: track 6.93 -> 32.4 mm
- net DATA_L2: track 8.07 -> 30.6 mm
- net Net-(R10-Pad1): track 0.00 -> 21.6 mm, vias 0 -> 1
- net LCD_RS: track 0.00 -> 20.2 mm
- net LCD_RW: track 0.00 -> 18.9 mm
- net DB3: track 0.00 -> 18.8 mm, vias 0 -> 1
- net D-: track 0.00 -> 16.3 mm
- net DB2: track 0.00 -> 16.3 mm, vias 0 -> 1
- net LCD_E: track 0.00 -> 14.3 mm
- net Net-(R15-Pad1): track 21.8 -> 8.66 mm
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Other:
- board size 70 x 62.5 mm -> 69.5 x 62.5 mm
